Commit message: code u5a2

File: src/u05/model/trike.xacro (robot description, xacro)
@@ -1,5 +1,4 @@
 <?xml version="1.0"?>
-<!-- Revolute-Revolute Manipulator -->
-<robot name="rrbot_model" xmlns:xacro="http://www.ros.org/wiki/xacro">
+<robot name="trike" xmlns:xacro="http://www.ros.org/wiki/xacro">
   <!-- Constants for robot dimensions -->
   <xacro:property name="PI" value="3.1415926535897931"/>
@@ -10,17 +9,15 @@
   <xacro:property name="wheel_l" value="0.1" />
   <!-- Import your model behavior in Gazebo -->
-  <xacro:include filename="$(find rrbot_description)/model/rrbot.gazebo.xacro" />
+  <xacro:include filename="$(find u05)/model/trike.gazebo" />
   <!-- Import Rviz colors -->
-  <xacro:include filename="$(find rrbot_description)/model/materials.xacro" />
-  <!-- Define your rrbot model -->
-  <xacro:macro name="rrbot" params="parent name *origin">
-  <!-- Propagate the name to all elements to make them unique -->
-  <joint name="${name}_fixed" type="fixed">
-    <insert_block name="origin"/>
-    <parent link="${parent}"/>
-    <child link="${name}_body"/>
+  <xacro:include filename="$(find rrbot_description)/urdf/materials.xacro" />
+  <!-- Connect to world -->
+  <link name="world"/>
+  <joint name="fixed" type="fixed">
+    <parent link="world"/>
+    <child link="body"/>
   </joint>
   <!-- Body -->
-  <link name="${name}_body">
+  <link name="body">
     <visual>
       <origin xyz="0 0 ${2 * wheel_r}" rpy="0 0 0"/>
@@ -28,5 +25,5 @@
 	<box size="${body_w} ${body_l} ${body_h}"/>
       </geometry>
-      <material name="RRBOT/orange"/>
+      <material name="orange"/>
     </visual>
     <inertial>
@@ -37,5 +34,5 @@
   </link>
   <!-- Wheel Front -->
-  <link name="${name}_wheel_1">
+  <link name="wheel_1">
     <visual>
       <origin xyz="0 0 0" rpy="0 ${PI / 2} 0"/>
@@ -43,5 +40,5 @@
 	<cylinder radius="${wheel_r}" length="${wheel_l}"/>
       </geometry>
-      <material name="RRBOT/black"/>
+      <material name="black"/>
     </visual>
     <inertial>
@@ -51,13 +48,12 @@
     </inertial>
   </link>
-  <joint name="${name}_joint_1" type="continuous">
-    <parent link="${name}_body"/>
-    <child link="${name}_wheel_1"/>
+  <joint name="joint_1" type="fixed">
+    <parent link="body"/>
+    <child link="wheel_1"/>
     <origin xyz="0 ${-0.45 * body_l} ${wheel_r}" rpy="0 0 0"/>
     <axis xyz="0 1 0"/>
-    <limit effort="10" velocity="0.5"/>
   </joint>
   <!-- Wheel Rear 1 -->
-  <link name="${name}_wheel_2">
+  <link name="wheel_2">
     <visual>
       <origin xyz="${-wheel_l / 2} 0 0" rpy="0 ${PI / 2} 0"/>
@@ -65,5 +61,5 @@
         <cylinder radius="${wheel_r}" length="${wheel_l}"/>
       </geometry>
-      <material name="RRBOT/black"/>
+      <material name="black"/>
     </visual>
     <inertial>
@@ -73,13 +69,12 @@
     </inertial>
   </link>
-  <joint name="${name}_joint_2" type="continuous">
-    <parent link="${name}_body"/>
-    <child link="${name}_wheel_2"/>
+  <joint name="joint_2" type="fixed">
+    <parent link="body"/>
+    <child link="wheel_2"/>
     <origin xyz="${-body_w / 2} ${0.45 * body_l} ${wheel_r}" rpy="0 0 0"/>
     <axis xyz="0 1 0"/>
-    <limit effort="10" velocity="0.5"/>
   </joint>
   <!-- Wheel Rear 2 -->
-   <link name="${name}_wheel_3">
+   <link name="wheel_3">
     <visual>
       <origin xyz="${wheel_l / 2} 0 0" rpy="0 ${PI / 2} 0"/>
@@ -87,5 +82,5 @@
         <cylinder radius="${wheel_r}" length="${wheel_l}"/>
       </geometry>
-      <material name="RRBOT/black"/>
+      <material name="black"/>
     </visual>
     <inertial>
@@ -95,43 +90,60 @@
     </inertial>
   </link>
-  <joint name="${name}_joint_3" type="continuous">
-    <parent link="${name}_body"/>
-    <child link="${name}_wheel_3"/>
+  <joint name="joint_3" type="fixed">
+    <parent link="body"/>
+    <child link="wheel_3"/>
     <origin xyz="${body_w / 2} ${0.45 * body_l} ${wheel_r}" rpy="0 0 0"/>
     <axis xyz="0 1 0"/>
-    <limit effort="10" velocity="0.5"/>
   </joint>
- <transmission name="${name}_tran_1">
+  <!-- Camera -->
+  <link name="camera">
+    <visual>
+      <origin xyz="0 0 0" rpy="0 0 0"/>
+      <geometry>
+	<box size="0.1 0.1 0.1"/>
+      </geometry>
+      <material name="blue"/>
+    </visual>
+    <inertial>
+      <mass value="1e-5" />
+      <origin xyz="0 0 0" rpy="0 0 0"/>
+      <inertia ixx="1e-6" ixy="0" ixz="0" iyy="1e-6" iyz="0" izz="1e-6" />
+    </inertial>
+  </link>
+  <joint name="joint_camera" type="fixed">
+    <axis xyz="0 0 1" />
+    <origin xyz="0 ${-0.45 * body_l} ${body_h + wheel_r}" rpy="0 0 ${-PI / 2}"/>
+    <parent link="body"/>
+    <child link="camera"/>
+  </joint>
+  <!-- Hokuyo Laser -->
+  <link name="laser">
+    <visual>
+      <origin xyz="0 0 0" rpy="0 0 0"/>
+      <geometry>
+        <mesh filename="package://rrbot_description/meshes/hokuyo.dae"/>
+      </geometry>
+    </visual>
+    <inertial>
+      <mass value="1e-5" />
+      <origin xyz="0 0 0" rpy="0 0 0"/>
+      <inertia ixx="1e-6" ixy="0" ixz="0" iyy="1e-6" iyz="0" izz="1e-6" />
+    </inertial>
+  </link>
+  <joint name="joint_laser" type="fixed">
+    <axis xyz="0 0 1" />
+    <origin xyz="0 ${-0.45 * body_l} ${body_h + wheel_r + 0.1}" rpy="0 0 0"/>
+    <parent link="body"/>
+    <child link="laser"/>
+  </joint>
+  <transmission name="tran_1">
     <type>transmission_interface/SimpleTransmission</type>
-    <robotNamespace>${name}</robotNamespace>
-    <joint name="${name}_joint_1">
+    <joint name="joint_1">
       <hardwareInterface>PositionJointInterface</hardwareInterface>
     </joint>
-    <actuator name="${name}_motor_1">
+    <actuator name="motor_1">
+      <hardwareInterface>PositionJointInterface</hardwareInterface>
       <mechanicalReduction>1</mechanicalReduction>
     </actuator>
   </transmission>
-  <transmission name="${name}_tran_2">
-    <type>transmission_interface/SimpleTransmission</type>
-    <robotNamespace>${name}</robotNamespace>
-    <joint name="${name}_joint_2">
-      <hardwareInterface>PositionJointInterface</hardwareInterface>
-    </joint>
-    <actuator name="${name}_motor_2">
-      <mechanicalReduction>1</mechanicalReduction>
-    </actuator>
-  </transmission>
-  <transmission name="${name}_tran_3">
-    <type>transmission_interface/SimpleTransmission</type>
-    <robotNamespace>${name}</robotNamespace>
-    <joint name="${name}_joint_3">
-      <hardwareInterface>PositionJointInterface</hardwareInterface>
-    </joint>
-    <actuator name="${name}_motor_3">
-      <mechanicalReduction>1</mechanicalReduction>
-    </actuator>
-  </transmission>
-  <!-- Instance your model behavior in Gazebo keeping the name -->
-  <xacro:rrbot_gazebo name="${name}"/>
-  </xacro:macro>
 </robot>

Commit message: src << laser

File: src/u05/model/trike.xacro (robot description, xacro)
@@ -133,5 +133,5 @@
   <joint name="joint_laser" type="fixed">
     <axis xyz="0 0 1" />
-    <origin xyz="0 ${-0.45 * body_l} ${body_h + wheel_r + 0.1}" rpy="0 0 0"/>
+    <origin xyz="0 ${-0.45 * body_l} ${body_h + wheel_r + 0.1}" rpy="0 ${PI / 16} ${-PI / 2}"/>
     <parent link="body"/>
     <child link="laser"/>

Commit message: modell mit joints, die besagten fehler produzieren. viel spass beim debuggen. könnte irgendetwas mit der fehlenden tf zu tun haben.

File: src/u05/model/trike.xacro (robot description, xacro)
@@ -33,4 +33,25 @@
     </inertial>
   </link>
+  <!-- Front Axis (yaw) -->
+  <link name="axis">
+    <visual>
+      <origin xyz="0 0 0" rpy="0 0 0"/>
+      <geometry>
+	<box size="0.01 0.01 0.01"/>
+      </geometry>
+    </visual>
+    <inertial>
+      <mass value="0.01" />
+      <origin xyz="0 0 0" rpy="0 0 0"/>
+      <inertia ixx="1e-6" ixy="1e-6" ixz="1e-6" iyy="1e-6" iyz="1e-6" izz="1e-6" />
+    </inertial>
+  </link>
+  <joint name="joint_1" type="revolute">
+    <parent link="body"/>
+    <child link="axis"/>
+    <origin xyz="0 ${-0.45 * body_l} ${wheel_r}" rpy="0 0 0"/>
+    <axis xyz="0 0 1"/>
+   <limit lower="${-PI / 2}" upper="${PI / 2}" effort="10" velocity="0.5" />
+  </joint>
   <!-- Wheel Front -->
   <link name="wheel_1">
@@ -48,8 +69,8 @@
     </inertial>
   </link>
-  <joint name="joint_1" type="fixed">
-    <parent link="body"/>
+  <joint name="joint_0" type="continuous">
+    <parent link="axis"/>
     <child link="wheel_1"/>
-    <origin xyz="0 ${-0.45 * body_l} ${wheel_r}" rpy="0 0 0"/>
+    <origin xyz="0 0 0" rpy="0 0 0"/>
     <axis xyz="0 1 0"/>
   </joint>

Commit message: fix für gelenke-reset: die inertials müssen sinnvoll gesetzt werden.

File: src/u05/model/trike.xacro (robot description, xacro)
@@ -30,5 +30,5 @@
       <mass value="1" />
       <origin xyz="0 0 0" rpy="0 0 0"/>
-      <inertia ixx="1e-6" ixy="1e-6" ixz="1e-6" iyy="1e-6" iyz="1e-6" izz="1e-6" />
+      <inertia ixx="1" ixy="0" ixz="0" iyy="1" iyz="0" izz="1" />
     </inertial>
   </link>
@@ -44,5 +44,5 @@
       <mass value="0.01" />
       <origin xyz="0 0 0" rpy="0 0 0"/>
-      <inertia ixx="1e-6" ixy="1e-6" ixz="1e-6" iyy="1e-6" iyz="1e-6" izz="1e-6" />
+      <inertia ixx="1" ixy="0" ixz="0" iyy="1" iyz="0" izz="1" />
     </inertial>
   </link>
@@ -52,5 +52,6 @@
     <origin xyz="0 ${-0.45 * body_l} ${wheel_r}" rpy="0 0 0"/>
     <axis xyz="0 0 1"/>
-   <limit lower="${-PI / 2}" upper="${PI / 2}" effort="10" velocity="0.5" />
+    <limit lower="${-PI / 2}" upper="${PI / 2}" effort="10" velocity="0.5" />
+    <dynamics damping="0.7" />
   </joint>
   <!-- Wheel Front -->
@@ -66,5 +67,5 @@
       <mass value="0.1" />
       <origin xyz="0 0 0" rpy="0 0 0"/>
-      <inertia ixx="1e-6" ixy="1e-6" ixz="1e-6" iyy="1e-6" iyz="1e-6" izz="1e-6" />
+      <inertia ixx="1" ixy="0" ixz="0" iyy="1" iyz="0" izz="1" />
     </inertial>
   </link>
@@ -74,4 +75,5 @@
     <origin xyz="0 0 0" rpy="0 0 0"/>
     <axis xyz="0 1 0"/>
+    <dynamics damping="0.7" />
   </joint>
   <!-- Wheel Rear 1 -->
@@ -87,5 +89,5 @@
       <mass value="0.1" />
       <origin xyz="0 0 ${wheel_r}" rpy="0 0 0"/>
-      <inertia ixx="1e-6" ixy="1e-6" ixz="1e-6" iyy="1e-6" iyz="1e-6" izz="1e-6" />
+      <inertia ixx="1" ixy="0" ixz="0" iyy="1" iyz="0" izz="1" />
     </inertial>
   </link>
@@ -108,5 +110,5 @@
       <mass value="0.1" />
       <origin xyz="0 0 ${wheel_r}" rpy="0 0 0"/>
-      <inertia ixx="1e-6" ixy="1e-6" ixz="1e-6" iyy="1e-6" iyz="1e-6" izz="1e-6" />
+      <inertia ixx="1" ixy="0" ixz="0" iyy="1" iyz="0" izz="1" />
     </inertial>
   </link>
@@ -129,5 +131,5 @@
       <mass value="1e-5" />
       <origin xyz="0 0 0" rpy="0 0 0"/>
-      <inertia ixx="1e-6" ixy="0" ixz="0" iyy="1e-6" iyz="0" izz="1e-6" />
+      <inertia ixx="1" ixy="0" ixz="0" iyy="1" iyz="0" izz="1" />
     </inertial>
   </link>
@@ -149,5 +151,5 @@
       <mass value="1e-5" />
       <origin xyz="0 0 0" rpy="0 0 0"/>
-      <inertia ixx="1e-6" ixy="0" ixz="0" iyy="1e-6" iyz="0" izz="1e-6" />
+      <inertia ixx="1" ixy="0" ixz="0" iyy="1" iyz="0" izz="1" />
     </inertial>
   </link>

Commit message: vorderachse lässt sich jetzt lenken

File: src/u05/model/trike.xacro (robot description, xacro)
@@ -47,5 +47,5 @@
     </inertial>
   </link>
-  <joint name="joint_1" type="revolute">
+  <joint name="joint_axis" type="revolute">
     <parent link="body"/>
     <child link="axis"/>
@@ -70,10 +70,9 @@
     </inertial>
   </link>
-  <joint name="joint_0" type="continuous">
+  <joint name="joint_1" type="fixed">
     <parent link="axis"/>
     <child link="wheel_1"/>
     <origin xyz="0 0 0" rpy="0 0 0"/>
     <axis xyz="0 1 0"/>
-    <dynamics damping="0.7" />
   </joint>
   <!-- Wheel Rear 1 -->
@@ -160,10 +159,10 @@
     <child link="laser"/>
   </joint>
-  <transmission name="tran_1">
+  <transmission name="tran_axis">
     <type>transmission_interface/SimpleTransmission</type>
-    <joint name="joint_1">
+    <joint name="joint_axis">
       <hardwareInterface>PositionJointInterface</hardwareInterface>
     </joint>
-    <actuator name="motor_1">
+    <actuator name="motor_axis">
       <hardwareInterface>PositionJointInterface</hardwareInterface>
       <mechanicalReduction>1</mechanicalReduction>
